File: KiCad/Miniaturazed_Two_Stage_transmitter/Miniaturazed_Two_Stage_transmitter.kicad_pcb (KiCad board)
At the start: 2 copper layers, 65.7 x 34.8 mm, 51 parts

Commit message: pcb cleanup
Parts:
- moved YC1 0.06 mm to (87.0, 70.8)
Connections:
- CA1 pad 2: 0 -> /Full/GNDA
- CA2 pad 2: 0 -> /Full/GNDA
- CA5 pad 2: 0 -> /Full/GNDA
- CB1 pad 2: 0 -> /Single_stage_transmitter/GNDB
- CB2 pad 2: 0 -> /Single_stage_transmitter/GNDB
- CB3 pad 2: 0 -> /Single_stage_transmitter/GNDB
- CC1 pad 2: 0 -> /Single_stage_transmitter/GNDC
- CC2 pad 2: 0 -> /Single_stage_transmitter/GNDC
- CC3 pad 2: 0 -> /Single_stage_transmitter/GNDC
- QB1 pad 3: 0 -> /Single_stage_transmitter/GNDB
- QC1 pad 3: 0 -> /Single_stage_transmitter/GNDC
- RA3 pad 2: 0 -> /Full/GNDA
- TP2 pad 1: 0 -> /Full/GNDA
- TPB2 pad 1: 0 -> /Single_stage_transmitter/GNDB
- V2 pad 2: 0 -> /Full/GNDA
- V3 pad 2: 0 -> /Single_stage_transmitter/GNDB
- V4 pad 2: 0 -> /Single_stage_transmitter/GNDC
- YA1 pad 3: 0 -> /Full/GNDA
- YB1 pad 3: 0 -> /Single_stage_transmitter/GNDB
- YC1 pad 3: 0 -> /Single_stage_transmitter/GNDC
Routing:
- net 0: track 103.0 -> 0.00 mm, vias 4 -> 0
- net /Full/GNDA: track 0.00 -> 57.5 mm, vias 0 -> 2
- net /Single_stage_transmitter/GNDB: track 0.00 -> 35.2 mm, vias 0 -> 2
- net /Single_stage_transmitter/GNDC: track 0.00 -> 10.3 mm

Commit message: added planning gantt chart
Other:
- board text added: "GND"
- board text added: "VCC"
