File: KiCad/Single_Stage_Transmitter/Single_Stage_Transmitter.kicad_sch (KiCad schematic)
At the start: 11 parts, among them Q1 QRF

Commit message: modified sst schematic
Parts:
- added AE1: Antenna, symbol Device:Antenna
- added C4: 580n, symbol Device:C
- added L2: 82n, symbol Device:L
- C1: value 2p -> 3p
- C2: value 10p -> 15p
- C3: value 34p -> 15p
- Cm1: value 1f -> 15f
- L1: value 50n -> 1u
- Lm1: value 1.126m -> 690u
- R1: value 150k -> 390k
- R2: value 0.5 -> 2.2Meg
- Rs1: value 50 -> 30
- V1: value PULSE(0 3 0 1n 1n 1) -> 3; footprint (none) -> Package_QFP:TQFP-44_10x10mm_P0.8mm
Connections:
- net 0: now also C4.2
- net OUT: now also C3.1, L1.1, AE1.1 (A), L2.2; no longer C1.1, C3.2, Q1.1 (C), R2.1, Rs1.2
- net Base: now reaches C1.2, C2.1, Lm1.1, Q1.2 (B), R1.2
- net at R2.2: now also V1.1, L2.1; no longer L1.2
- new net: C4.1, R1.1, R2.1
- new net Collector: C1.1, C3.2, L1.2, Q1.1 (C), Rs1.2
Other:
- note added: ".tran 100u 10m 0 100u"
- note removed: ".options reltol=1e-4 trtol=1"
- note removed: ".tran 0.2n 40u 0 0.2n"
- moved on the sheet: C2, C3, L1, Q1

Commit message: oscillation with own calculations
Parts:
- removed AE1: Antenna, symbol Device:Antenna
- added C5: 2p, symbol Device:C
- added C6: 10p, symbol Device:C
- added Rs2: 25, symbol Device:R
- C2: value 15p -> 10p
- C3: value 15p -> 6p
- C4: value 580n -> 0.5n
- Cm1: value 15f -> 22.22f
- L1: renamed from L2; value 82n -> 600n
- L2: renamed from L1; value 1u -> 220n
- Lm1: value 690u -> 54u
- R1: value 390k -> 50k
- R2: value 2.2Meg -> 50k
- Rs1: value 30 -> 50
Connections:
- net 0: now also C6.2, Rs2.1
- net Collector: now also C6.1
- net OUT: now also C5.1
- net Vcc: now reaches L1.1, R2.2, V1.1
- new net: C5.2, Rs2.2
Other:
- note added: ".tran 100p 150u 0 100p .ic V(Net-_C4-Pad1_)=1.9 V(/Base)=0.8 .model __Q1 NPN(BF=100 IS=1e-16 VAF=100 CJE=1p CJC=0.5p TF=20p)"
- note added: "5.4mH 0.2222f"
- note removed: ".tran 100u 10m 0 100u"

Commit message: improved oscillation with better values
Parts:
- C6: value 10p -> 4p
Other:
- note added: ".tran 500p 5m 0 UIC .ic V(Net-_C4-Pad1_)=1.9 V(/Base)=0.8 .model __Q1 NPN(BF=100 IS=1e-16 VAF=100 CJE=1p CJC=0.5p TF=20p) .option method=trap .option trtol=3 .option reltol=0.003 .option abstol=1nA vntol=1mV .option trtol=7 .save v(OUT) v(/Base) v(Net-_C4-Pad1_)"
- note removed: ".tran 100p 150u 0 100p .ic V(Net-_C4-Pad1_)=1.9 V(/Base)=0.8 .model __Q1 NPN(BF=100 IS=1e-16 VAF=100 CJE=1p CJC=0.5p TF=20p)"
Changed lines of the file:
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@@
 		)
 	)
-	(text ".tran 100p 150u 0 100p\n.ic V(Net-_C4-Pad1_)=1.9 V(/Base)=0.8\n.model __Q1 NPN(BF=100 IS=1e-16 VAF=100 CJE=1p CJC=0.5p TF=20p)\n"
+	(text ".tran 500p 5m 0 UIC\n\n.ic V(Net-_C4-Pad1_)=1.9 V(/Base)=0.8\n.model __Q1 NPN(BF=100 IS=1e-16 VAF=100 CJE=1p CJC=0.5p TF=20p)\n\n.option method=trap\n.option trtol=3\n.option reltol=0.003\n.option abstol=1nA vntol=1mV\n.option trtol=7\n\n.save v(OUT) v(/Base) v(Net-_C4-Pad1_)\n"
 		(exclude_from_sim no)
-		(at 88.9 90.932 0)
+		(at 56.896 107.696 0)
 		(effects
 			(font
 				(size 1.27 1.27)
 			)
+			(justify left)
 		)
 	)
@@
 			)
 		)
-		(property "Value" "10p"
+		(property "Value" "4p"
 			(at 145.796 78.232 0)
 			(show_name no)

Commit message: recalculation to remove collector capacitor
Parts:
- removed C6: 4p, symbol Device:C
- added R3: 0, symbol Device:R
- C2: value 10p -> 5p
- C4: value 0.5n -> 580n
- L1: value 600n -> 200n
- L2: value 220n -> 298n
- R2: value 50k -> 200k
Connections:
- net Vcc: now also R3.2; no longer L1.1, R2.2
- new net: L1.1, R2.2, R3.1
Other:
- note added: ".tran 500p 300u 0 500p .save v(/OUT) v(/Base) v(/Collector)"
- note removed: ".tran 500p 5m 0 UIC .ic V(Net-_C4-Pad1_)=1.9 V(/Base)=0.8 .model __Q1 NPN(BF=100 IS=1e-16 VAF=100 CJE=1p CJC=0.5p TF=20p) .option method=trap .option trtol=3 .option reltol=0.003 .option abstol=1nA vntol=1mV .option trtol=7 .save v(OUT) v(/Base) v(Net-_C4-Pad1_)"
Changed lines of the file:
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@@
 	(text "5.4mH\n0.2222f\n"
 		(exclude_from_sim no)
-		(at 105.41 49.022 0)
+		(at 103.378 46.228 0)
 		(effects
 			(font
@@
 		)
 	)
-	(text ".tran 500p 5m 0 UIC\n\n.ic V(Net-_C4-Pad1_)=1.9 V(/Base)=0.8\n.model __Q1 NPN(BF=100 IS=1e-16 VAF=100 CJE=1p CJC=0.5p TF=20p)\n\n.option method=trap\n.option trtol=3\n.option reltol=0.003\n.option abstol=1nA vntol=1mV\n.option trtol=7\n\n.save v(OUT) v(/Base) v(Net-_C4-Pad1_)\n"
+	(text ".tran 500p 300u 0 500p\n\n.save v(/OUT) v(/Base) v(/Collector)"
 		(exclude_from_sim no)
-		(at 56.896 107.696 0)
+		(at 57.15 96.012 0)
 		(effects
 			(font
@@
 	)
 	(junction
-		(at 142.24 85.09)
-		(diameter 0)
-		(color 0 0 0 0)
-	)
-	(junction
 		(at 132.08 85.09)
 		(diameter 0)
@@
 	)
 	(junction
-		(at 142.24 63.5)
-		(diameter 0)
-		(color 0 0 0 0)
-	)
-	(junction
 		(at 142.24 50.8)
 		(diameter 0)
@@
 	(wire
 		(pts
-			(xy 57.15 39.37) (xy 74.93 39.37)
+			(xy 57.15 39.37) (xy 62.23 39.37)
 		)
 		(stroke
@@
 	(wire
 		(pts
-			(xy 142.24 63.5) (xy 142.24 72.39)
-		)
-		(stroke
-			(width 0)
-			(type default)
-		)
-	)
-	(wire
-		(pts
 			(xy 106.68 59.69) (xy 109.22 59.69)
 		)
@@
 	(wire
 		(pts
+			(xy 69.85 39.37) (xy 74.93 39.37)
+		)
+		(stroke
+			(width 0)
+			(type default)
+		)
+	)
+	(wire
+		(pts
 			(xy 116.84 67.31) (xy 129.54 67.31)
 		)
@@
 	(wire
 		(pts
-			(xy 142.24 80.01) (xy 142.24 85.09)
-		)
-		(stroke
-			(width 0)
-			(type default)
-		)
-	)
-	(wire
-		(pts
 			(xy 142.24 48.26) (xy 142.24 50.8)
 		)
@@
 	(wire
 		(pts
-			(xy 142.24 85.09) (xy 153.67 85.09)
+			(xy 132.08 85.09) (xy 153.67 85.09)
 		)
 		(stroke
@@
 		(pts
 			(xy 64.77 85.09) (xy 64.77 88.9)
-		)
-		(stroke
-			(width 0)
-			(type default)
-		)
-	)
-	(wire
-		(pts
-			(xy 132.08 85.09) (xy 142.24 85.09)
 		)
 		(stroke
@@
 	)
 	(symbol
-		(lib_id "Device:C")
-		(at 142.24 76.2 0)
+		(lib_id "Device:R")
+		(at 66.04 39.37 270)
 		(unit 1)
 		(body_style 1)
@@
 		(in_pos_files yes)
 		(dnp no)
-		(property "Reference" "C6"
-			(at 145.542 76.454 0)
-			(show_name no)
-			(do_not_autoplace no)
-			(effects
-				(font
-					(size 1.27 1.27)
-				)
-				(justify left)
-			)
-		)
-		(property "Value" "4p"
-			(at 145.796 78.232 0)
-			(show_name no)
-			(do_not_autoplace no)
-			(effects
-				(font
-					(size 1.27 1.27)
-				)
-				(justify left)
+		(fields_autoplaced yes)
+		(property "Reference" "R3"
+			(at 66.04 33.02 90)
+			(show_name no)
+			(do_not_autoplace no)
+			(effects
+				(font
+					(size 1.27 1.27)
+				)
+			)
+		)
+		(property "Value" "0"
+			(at 66.04 35.56 90)
+			(show_name no)
+			(do_not_autoplace no)
+			(effects
+				(font
+					(size 1.27 1.27)
+				)
 			)
 		)
 		(property "Footprint" ""
-			(at 143.2052 80.01 0)
+			(at 66.04 37.592 90)
 			(hide yes)
 			(show_name no)
@@
 		)
 		(property "Datasheet" ""
-			(at 142.24 76.2 0)
-			(hide yes)
-			(show_name no)
-			(do_not_autoplace no)
-			(effects
-				(font
-					(size 1.27 1.27)
-				)
-			)
-		)
-		(property "Description" "Unpolarized capacitor"
-			(at 142.24 76.2 0)
-			(hide yes)
-			(show_name no)
-			(do_not_autoplace no)
-			(effects
-				(font
-					(size 1.27 1.27)
-				)
-			)
+			(at 66.04 39.37 0)
+			(hide yes)
+			(show_name no)
+			(do_not_autoplace no)
+			(effects
+				(font
+					(size 1.27 1.27)
+				)
+			)
+		)
+		(property "Description" "Resistor"
+			(at 66.04 39.37 0)
+			(hide yes)
+			(show_name no)
+			(do_not_autoplace no)
+			(effects
+				(font
+					(size 1.27 1.27)
+				)
+			)
+		)
+		(pin "2"
 		)
 		(pin "1"
-		)
-		(pin "2"
 		)
 		(instances
 			(project "Single_Stage_Transmitter"
 				(path "/2688bd9c-c39c-4a29-8195-973e7622281f"
-					(reference "C6")
+					(reference "R3")
 					(unit 1)
 				)
@@
 			)
 		)
-		(property "Value" "600n"
+		(property "Value" "200n"
 			(at 143.51 45.7199 0)
 			(show_name no)
@@
 			)
 		)
-		(property "Value" "50k"
+		(property "Value" "200k"
 			(at 77.47 60.9599 0)
 			(show_name no)
@@
 			)
 		)
-		(property "Value" "0.5n"
+		(property "Value" "580n"
 			(at 78.74 81.2799 0)
 			(show_name no)
@@
 			)
 		)
-		(property "Value" "220n"
+		(property "Value" "298n"
 			(at 143.51 58.4199 0)
 			(show_name no)
@@
 			)
 		)
-		(property "Value" "10p"
+		(property "Value" "5p"
 			(at 122.936 82.042 0)
 			(show_name no)
